Commit message: costmap node

File: src/gazebo/launch/env.urdf (robot description, URDF)
Before this commit: robot robot, 11 links, 11 joints
Links:
- removed link box1
- removed link box2
- removed link box3
- removed link box4
- removed link box5
- removed link cyl1
- removed link cyl2
- removed link wall
- removed link wall1
- removed link wall2
- removed link wall3
- added link box1_link; visual box size=3 3 3.0
- added link box2_link; visual box size=3 3 3.0
- added link box3_link; visual box size=3 3 3.0
- added link box4_link; visual box size=2 2 3.0
- added link box5_link; visual box size=2 2 3.0
- added link cyl1_link; visual cylinder length=3 radius=3
- added link cyl2_link; visual cylinder length=3 radius=2
- added link sim_world
- added link wall1_link; visual box size=30 0.5 3.0
- added link wall2_link; visual box size=30 0.5 3.0
- added link wall3_link; visual box size=0.5 30 3.0
- added link wall4_link; visual box size=0.5 30 3.0
Joints:
- removed joint j1
- removed joint j10
- removed joint j11
- removed joint j2
- removed joint j3
- removed joint j4
- removed joint j5
- removed joint j6
- removed joint j7
- removed joint j8
- removed joint j9
- added joint box1_joint: type fixed, parent sim_world, child box1_link, origin xyz=7 -6 0
- added joint box2_joint: type fixed, parent sim_world, child box2_link, origin xyz=-8 6 0
- added joint box3_joint: type fixed, parent sim_world, child box3_link, origin xyz=4 9 0
- added joint box4_joint: type fixed, parent sim_world, child box4_link, origin xyz=9 3 0
- added joint box5_joint: type fixed, parent sim_world, child box5_link, origin xyz=1 -10 0
- added joint cyl1_joint: type fixed, parent sim_world, child cyl1_link, origin xyz=0 0 0
- added joint cyl2_joint: type fixed, parent sim_world, child cyl2_link, origin xyz=-7 -7 0
- added joint wall1_joint: type fixed, parent sim_world, child wall1_link, origin xyz=0 -15 0
- added joint wall2_joint: type fixed, parent sim_world, child wall2_link, origin xyz=0 15 0
- added joint wall3_joint: type fixed, parent sim_world, child wall3_link, origin xyz=15 0 0
- added joint wall4_joint: type fixed, parent sim_world, child wall4_link, origin xyz=-15 0 0
